File: hardware/kicad/thumbsup.kicad_pcb (KiCad board)
At the start: 2 copper layers, 0 parts

Commit message: hardware: generated PCB layout pipeline (mech outline, placement, copper, Freerouting), rev v1.2
- tools/mech/chassis.py: Bambu 3MF -> PCB bay outline, boss positions, fit check
- tools/pcb/: board builder (netlist -> pcbnew), obstacle-aware placement with
  0 placement problems, power pours / via fields / gate and Kelvin stubs, pickup
  and GND vias, Freerouting DSN/SES driver, JLC fab outputs
- circuit: J4/C4/C426 dropped, motor holes between the FET rows, Kelvin net-ties
  in the shunt pad gap, M2.5 holes, SWD pad rows, fewer test points, I_x+ named
- docs: LAYOUT.md rewritten for the generated layout, PARTS/REQUIREMENTS/REVIEW
  updated; routing status recorded in LAYOUT.md section 5 (102 unconnected left,
  board is over-dense for a fully automatic finish)

Co-Authored-By: Claude Fable 5.1 <noreply@anthropic.com>
Parts:
- added A1: Pico W, RaspberryPi_Pico_W_SMD_HandSolder, F.Cu at (67.7, 25.4)
- added C1: 10u 50V, C_1206_3216Metric, B.Cu at (9.54, 10.8)
- added C10: 10u 50V, C_1206_3216Metric, B.Cu at (59.7, 25.0)
- added C11: 10u 50V, C_1206_3216Metric, B.Cu at (64.7, 25.0)
- added C12: 100n 50V, C_0603_1608Metric, B.Cu at (68.8, 24.6)
- added C13: 100n 50V, C_0603_1608Metric, B.Cu at (72.1, 24.6)
- added C14: 22u 25V, C_0805_2012Metric, B.Cu at (75.6, 24.8)
- added C15: 22u 25V, C_0805_2012Metric, B.Cu at (59.1, 27.5)
- added C16: 1u 50V, C_0603_1608Metric, B.Cu at (70.6, 27.2)
- added C17: 10u 25V, C_0805_2012Metric, B.Cu at (74.1, 27.5)
- added C18: 1u 50V, C_0603_1608Metric, B.Cu at (58.9, 30.5)
- added C19: 10u 25V, C_0805_2012Metric, B.Cu at (62.8, 30.7)
- added C2: 10u 50V, C_1206_3216Metric, B.Cu at (5.34, 15.7)
- added C20: 100n, C_0402_1005Metric, B.Cu at (78.2, 41.8)
- added C200: 4.7u, C_0603_1608Metric, B.Cu at (39.5, 25.1)
- added C201: 100n, C_0402_1005Metric, B.Cu at (42.2, 24.8)
- added C202: 100n, C_0402_1005Metric, B.Cu at (44.4, 24.8)
- added C203: 1u, C_0402_1005Metric, B.Cu at (46.5, 24.8)
- added C204: 100n, C_0402_1005Metric, B.Cu at (48.7, 24.8)
- added C205: 100n, C_0402_1005Metric, B.Cu at (50.9, 24.8)
- added C206: 100n, C_0402_1005Metric, B.Cu at (36.8, 26.6)
- added C207: 10n, C_0402_1005Metric, B.Cu at (38.9, 26.6)
- added C208: 100n, C_0402_1005Metric, B.Cu at (41.1, 26.6)
- added C209: 10u 25V, C_0805_2012Metric, B.Cu at (44.0, 27.1)
- added C21: 100n, C_0402_1005Metric, B.Cu at (77.1, 44.4)
- added C210: 100n 50V, C_0603_1608Metric, B.Cu at (47.5, 26.9)
- added C220: 100n 50V, C_0603_1608Metric, B.Cu at (41.4, 8.44)
- added C221: 100n 50V, C_0603_1608Metric, B.Cu at (44.7, 8.44)
- added C222: 100n 50V, C_0603_1608Metric, B.Cu at (55.1, 23.3)
- added C223: 10u 50V, C_1206_3216Metric, B.Cu at (54.9, 15.2)
- added C224: 10u 50V, C_1206_3216Metric, B.Cu at (54.9, 20.0)
- added C225: 470u 25V hybrid, CP_Elec_10x10.5, F.Cu at (37.9, 5.60)
- added C23: 100n, C_0402_1005Metric, F.Cu at (11.0, 27.9)
- added C24: 100n, C_0402_1005Metric, F.Cu at (51.9, 42.3)
- added C25: 100n, C_0402_1005Metric, F.Cu at (11.0, 29.1)
- added C3: 100n 50V, C_0603_1608Metric, B.Cu at (8.72, 13.0)
- added C30: 100n, C_0402_1005Metric, B.Cu at (49.5, 9.95)
- added C300: 4.7u, C_0603_1608Metric, B.Cu at (82.6, 20.6)
- added C301: 100n, C_0402_1005Metric, B.Cu at (93.0, 20.3)
- added C302: 100n, C_0402_1005Metric, B.Cu at (95.2, 20.3)
- added C303: 1u, C_0402_1005Metric, B.Cu at (82.0, 22.1)
- added C304: 100n, C_0402_1005Metric, B.Cu at (84.2, 22.1)
- added C305: 100n, C_0402_1005Metric, B.Cu at (93.0, 22.1)
- added C306: 100n, C_0402_1005Metric, B.Cu at (80.6, 23.4)
- added C307: 10n, C_0402_1005Metric, B.Cu at (82.7, 23.4)
- added C308: 100n, C_0402_1005Metric, B.Cu at (93.0, 23.4)
- added C309: 10u 25V, C_0805_2012Metric, B.Cu at (81.3, 27.5)
- added C31: 100n, C_0402_1005Metric, B.Cu at (51.6, 9.95)
- added C310: 100n 50V, C_0603_1608Metric, B.Cu at (90.3, 14.8)
- added C320: 100n 50V, C_0603_1608Metric, B.Cu at (58.9, 35.2)
- added C321: 100n 50V, C_0603_1608Metric, B.Cu at (62.2, 35.2)
- added C322: 100n 50V, C_0603_1608Metric, B.Cu at (65.5, 35.2)
- added C323: 10u 50V, C_1206_3216Metric, B.Cu at (83.1, 25.2)
- added C324: 10u 50V, C_1206_3216Metric, B.Cu at (94.2, 25.2)
- added C325: 470u 25V hybrid, CP_Elec_10x10.5, F.Cu at (86.3, 31.9)
- added C40: 100n, C_0402_1005Metric, B.Cu at (47.7, 33.0)
- added C400: 4.7u, C_0603_1608Metric, B.Cu at (15.8, 35.7)
- added C401: 100n, C_0402_1005Metric, B.Cu at (20.3, 35.4)
- added C402: 100n, C_0402_1005Metric, B.Cu at (22.4, 35.4)
- added C403: 1u, C_0402_1005Metric, B.Cu at (27.1, 35.4)
- added C404: 100n, C_0402_1005Metric, B.Cu at (31.5, 36.1)
- added C405: 100n, C_0402_1005Metric, B.Cu at (33.6, 36.1)
- added C406: 100n, C_0402_1005Metric, B.Cu at (58.7, 38.2)
- added C407: 10n, C_0402_1005Metric, B.Cu at (50.3, 41.9)
- added C408: 100n, C_0402_1005Metric, B.Cu at (52.5, 41.9)
- added C409: 10u 25V, C_0805_2012Metric, B.Cu at (55.4, 42.5)
- added C41: 100n, C_0402_1005Metric, B.Cu at (36.8, 24.8)
- added C410: 100n 50V, C_0603_1608Metric, B.Cu at (58.9, 42.2)
- added C420: 100n 50V, C_0603_1608Metric, B.Cu at (41.8, 46.8)
- added C421: 100n 50V, C_0603_1608Metric, B.Cu at (45.1, 46.8)
- added C422: 100n 50V, C_0603_1608Metric, B.Cu at (48.4, 46.8)
- added C423: 10u 50V, C_1206_3216Metric, B.Cu at (15.6, 19.3)
- added C424: 10u 50V, C_1206_3216Metric, B.Cu at (27.3, 19.3)
- added C425: 470u 25V polymer 4A, CP_Elec_10x12.5, F.Cu at (50.5, 6.80)
- added C5: 10u 50V, C_1206_3216Metric, B.Cu at (8.00, 18.3)
- added C50: 100n, C_0402_1005Metric, B.Cu at (80.6, 7.88)
- added C51: 100n, C_0402_1005Metric, B.Cu at (82.7, 7.88)
- added C60: 100n, C_0402_1005Metric, B.Cu at (31.5, 21.8)
- added C61: 100n, C_0402_1005Metric, B.Cu at (33.6, 21.8)
- added C70: 100n, C_0402_1005Metric, B.Cu at (62.2, 7.49)
- added C71: 100n, C_0402_1005Metric, B.Cu at (64.4, 7.49)
- added C72: 1u, C_0402_1005Metric, B.Cu at (70.4, 7.49)
- added C73: 100n, C_0402_1005Metric, B.Cu at (72.5, 7.49)
- added C80: 100n, C_0402_1005Metric, B.Cu at (71.7, 13.3)
- added C81: 100n, C_0402_1005Metric, B.Cu at (76.0, 49.5)
- added C82: 100n, C_0402_1005Metric, F.Cu at (51.9, 43.6)
- added C83: 100n, C_0402_1005Metric, F.Cu at (101.5, 16.6)
- added D1: SMBJ15A, D_SMB, B.Cu at (23.3, 2.90)
- added D2: MMSZ5242B 12V, D_SOD-123, B.Cu at (8.74, 24.7)
- added D20: 1N5819WS, D_SOD-323, B.Cu at (39.1, 31.2)
- added D21: 1N5819WS, D_SOD-323, B.Cu at (44.1, 31.2)
- added D22: 1N5819WS, D_SOD-323, B.Cu at (37.9, 8.65)
- added D3: 1N5819WS, D_SOD-323, B.Cu at (67.2, 27.4)
- added D30: 1N5819WS, D_SOD-323, B.Cu at (100.2, 23.3)
- added D31: 1N5819WS, D_SOD-323, B.Cu at (100.2, 25.5)
- added D32: 1N5819WS, D_SOD-323, B.Cu at (62.7, 33.2)
- added D4: RED PWR, LED_0603_1608Metric, F.Cu at (10.6, 26.1)
- added D40: 1N5819WS, D_SOD-323, B.Cu at (56.4, 44.7)
- added D41: 1N5819WS, D_SOD-323, B.Cu at (34.8, 47.0)
- added D42: 1N5819WS, D_SOD-323, B.Cu at (38.4, 47.0)
- added D5: SK6812MINI-C, LED_SK6812MINI_PLCC4_3.5x3.5mm_P1.75mm, F.Cu at (9.60, 17.9)
- added D6: SK6812MINI-C, LED_SK6812MINI_PLCC4_3.5x3.5mm_P1.75mm, F.Cu at (9.60, 22.9)
- added FID1: Fiducial, Fiducial_1mm_Mask2mm, F.Cu at (11.0, 36.1)
- added FID2: Fiducial, Fiducial_1mm_Mask2mm, F.Cu at (47.3, 49.0)
- added FID3: Fiducial, Fiducial_1mm_Mask2mm, F.Cu at (99.7, 25.7)
- added H1: M2.5, MountingHole_2.7mm_M2.5, F.Cu at (3.70, 18.8)
- added H2: M2.5, MountingHole_2.7mm_M2.5, F.Cu at (101.5, 20.5)
- added H3: M2.5, MountingHole_2.7mm_M2.5, F.Cu at (52.8, 47.3)
- added J1: XT30PW-M, AMASS_XT30PW-M_1x02_P2.50mm_Horizontal, F.Cu at (26.3, 13.6)
- added J2: ARM link, PinHeader_1x02_P2.54mm_Vertical, F.Cu at (4.90, 24.8)
- added J20: SWD, SWD_1x05_P1.27mm_Pads, F.Cu at (36.8, 46.2)
- added J21: MOTOR L, MotorHoles_1x03_P5.90mm, F.Cu at (44.6, 22.2)
- added J3: EXPANSION, PinHeader_2x06_P2.54mm_Vertical, F.Cu at (35.2, 42.0)
- added J30: SWD, SWD_1x05_P1.27mm_Pads, F.Cu at (44.1, 46.2)
- added J31: MOTOR R, MotorHoles_1x03_P5.90mm, F.Cu at (88.5, 17.7)
- added J40: SWD, SWD_1x05_P1.27mm_Pads, F.Cu at (36.8, 49.0)
- added J41: MOTOR W, MotorHoles_1x03_P5.90mm, F.Cu at (21.4, 26.1)
- added L1: 4.7uH 4.9A, L_Changjiang_FNR4020S, B.Cu at (67.8, 21.3)
- added NT1: Kelvin, NetTie-2_Kelvin_0.4mm, B.Cu at (23.8, 7.30)
- added NT2: Kelvin, NetTie-2_Kelvin_0.4mm, B.Cu at (23.8, 9.70)
- added NT20: Kelvin, NetTie-2_Kelvin_0.4mm, F.Cu at (50.4, 32.3)
- added NT21: Kelvin, NetTie-2_Kelvin_0.4mm, F.Cu at (50.4, 34.7)
- added NT30: Kelvin, NetTie-2_Kelvin_0.4mm, F.Cu at (84.5, 3.20)
- added NT31: Kelvin, NetTie-2_Kelvin_0.4mm, F.Cu at (84.5, 5.60)
- added NT40: Kelvin, NetTie-2_Kelvin_0.4mm, F.Cu at (31.7, 31.5)
- added NT41: Kelvin, NetTie-2_Kelvin_0.4mm, F.Cu at (34.1, 31.5)
- added Q1: AP40P05, SOT-23, B.Cu at (7.62, 21.5)
- added Q20: HYG015N04LS1C2, PQFN-8-EP_6x5mm_P1.27mm_Generic, F.Cu at (38.8, 17.4)
- added Q21: HYG015N04LS1C2, PQFN-8-EP_6x5mm_P1.27mm_Generic, F.Cu at (38.8, 27.0)
- added Q22: HYG015N04LS1C2, PQFN-8-EP_6x5mm_P1.27mm_Generic, F.Cu at (44.6, 17.4)
- added Q23: HYG015N04LS1C2, PQFN-8-EP_6x5mm_P1.27mm_Generic, F.Cu at (44.6, 27.0)
- added Q24: HYG015N04LS1C2, PQFN-8-EP_6x5mm_P1.27mm_Generic, F.Cu at (50.5, 17.4)
- added Q25: HYG015N04LS1C2, PQFN-8-EP_6x5mm_P1.27mm_Generic, F.Cu at (50.5, 27.0)
- added Q30: HYG015N04LS1C2, PQFN-8-EP_6x5mm_P1.27mm_Generic, F.Cu at (82.5, 22.5)
- added Q31: HYG015N04LS1C2, PQFN-8-EP_6x5mm_P1.27mm_Generic, F.Cu at (82.5, 12.9)
- added Q32: HYG015N04LS1C2, PQFN-8-EP_6x5mm_P1.27mm_Generic, F.Cu at (88.5, 22.5)
- added Q33: HYG015N04LS1C2, PQFN-8-EP_6x5mm_P1.27mm_Generic, F.Cu at (88.5, 12.9)
- added Q34: HYG015N04LS1C2, PQFN-8-EP_6x5mm_P1.27mm_Generic, F.Cu at (94.3, 22.5)
- added Q35: HYG015N04LS1C2, PQFN-8-EP_6x5mm_P1.27mm_Generic, F.Cu at (94.3, 12.9)
- added Q40: HYG015N04LS1C2, PQFN-8-EP_6x5mm_P1.27mm_Generic, F.Cu at (15.6, 21.3)
- added Q41: HYG015N04LS1C2, PQFN-8-EP_6x5mm_P1.27mm_Generic, F.Cu at (15.6, 30.9)
- added Q42: HYG015N04LS1C2, PQFN-8-EP_6x5mm_P1.27mm_Generic, F.Cu at (21.4, 21.3)
- added Q43: HYG015N04LS1C2, PQFN-8-EP_6x5mm_P1.27mm_Generic, F.Cu at (21.4, 30.9)
- added Q44: HYG015N04LS1C2, PQFN-8-EP_6x5mm_P1.27mm_Generic, F.Cu at (27.4, 21.3)
- added Q45: HYG015N04LS1C2, PQFN-8-EP_6x5mm_P1.27mm_Generic, F.Cu at (27.4, 30.9)
- added Q46: AP40P05, SOT-23, B.Cu at (20.2, 20.1)
- added Q47: AO3400A, SOT-23, B.Cu at (33.1, 24.3)
- added Q48: AO3400A, SOT-23, B.Cu at (33.1, 33.6)
- added Q49: AO3400A, SOT-23, B.Cu at (51.3, 39.4)
- added Q50: AO3400A, SOT-23, B.Cu at (55.5, 39.4)
- added R1: 100k, R_0402_1005Metric, B.Cu at (18.0, 14.5)
- added R10: 100k, R_0402_1005Metric, B.Cu at (62.1, 27.0)
- added R11: 27k, R_0402_1005Metric, B.Cu at (64.3, 27.0)
- added R12: 100k, R_0402_1005Metric, B.Cu at (65.8, 30.2)
- added R13: 22k, R_0402_1005Metric, B.Cu at (76.0, 41.9)
- added R14: 10k, R_0402_1005Metric, B.Cu at (76.0, 43.1)
- added R15: 10k, R_0402_1005Metric, B.Cu at (78.2, 43.1)
- added R16: 1k, R_0402_1005Metric, B.Cu at (76.0, 45.7)
- added R2: 1mΩ 3W, R_2512_Shunt_Kelvin, B.Cu at (23.8, 8.50)
- added R20: 2.2k, R_0402_1005Metric, F.Cu at (11.0, 30.4)
- added R200: 10k, R_0402_1005Metric, B.Cu at (50.3, 26.6)
- added R201: 10k DNP, R_0402_1005Metric, B.Cu at (52.5, 26.6)
- added R202: 100k, R_0402_1005Metric, B.Cu at (36.8, 28.9)
- added R203: 10k, R_0402_1005Metric, B.Cu at (39.0, 28.9)
- added R204: 1k, R_0402_1005Metric, B.Cu at (41.2, 28.9)
- added R205: 10k, R_0402_1005Metric, B.Cu at (53.9, 11.2)
- added R206: 10k, R_0402_1005Metric, B.Cu at (49.5, 12.5)
- added R207: 10k, R_0402_1005Metric, B.Cu at (51.7, 12.5)
- added R208: 3.3k, R_0402_1005Metric, B.Cu at (76.0, 38.0)
- added R209: 3.3k, R_0402_1005Metric, B.Cu at (78.2, 38.0)
- added R21: 2.2k, R_0402_1005Metric, F.Cu at (11.0, 31.6)
- added R210: 3.3k, R_0402_1005Metric, B.Cu at (76.0, 39.3)
- added R211: 10k, R_0402_1005Metric, B.Cu at (78.2, 39.3)
- added R212: 10k, R_0402_1005Metric, B.Cu at (76.0, 40.6)
- added R213: 10k, R_0402_1005Metric, B.Cu at (78.2, 40.6)
- added R22: 10k, R_0402_1005Metric, F.Cu at (11.0, 32.9)
- added R220: 10, R_0402_1005Metric, B.Cu at (37.3, 10.4)
- added R221: 10, R_0402_1005Metric, B.Cu at (39.5, 10.4)
- added R222: 10, R_0402_1005Metric, B.Cu at (41.7, 10.4)
- added R223: 10, R_0402_1005Metric, B.Cu at (43.9, 10.4)
- added R224: 10, R_0402_1005Metric, B.Cu at (46.1, 10.4)
- added R225: 10, R_0402_1005Metric, B.Cu at (54.6, 24.8)
- added R226: 10k, R_0402_1005Metric, B.Cu at (54.6, 26.1)
- added R227: 10k, R_0402_1005Metric, B.Cu at (54.6, 27.4)
- added R228: 10k, R_0402_1005Metric, B.Cu at (54.6, 28.7)
- added R229: 10k, R_0402_1005Metric, B.Cu at (53.8, 9.96)
- added R23: 3.3k, R_0402_1005Metric, F.Cu at (11.0, 34.1)
- added R230: 10k, R_0402_1005Metric, B.Cu at (49.5, 11.2)
- added R231: 10k, R_0402_1005Metric, B.Cu at (51.7, 11.2)
- added R232: 2.2, R_0603_1608Metric, B.Cu at (43.9, 29.2)
- added R233: 2.2, R_0603_1608Metric, B.Cu at (47.2, 29.2)
- added R234: 2.2, R_0603_1608Metric, B.Cu at (50.5, 29.2)
- added R235: 1mΩ 3W, R_2512_Shunt_Kelvin, F.Cu at (50.4, 33.5)
- added R24: 100, R_0402_1005Metric, F.Cu at (51.9, 38.4)
- added R25: 100, R_0402_1005Metric, F.Cu at (51.9, 39.7)
- added R26: 100, R_0402_1005Metric, F.Cu at (51.9, 41.0)
- added R30: 10, R_0402_1005Metric, B.Cu at (11.5, 12.8)
- added R300: 10k, R_0402_1005Metric, B.Cu at (93.1, 14.6)
- added R301: 10k DNP, R_0402_1005Metric, B.Cu at (95.3, 14.6)
- added R302: 100k, R_0402_1005Metric, B.Cu at (86.6, 14.8)
- added R303: 10k, R_0402_1005Metric, B.Cu at (84.3, 27.0)
- added R304: 1k, R_0402_1005Metric, B.Cu at (86.5, 27.0)
- added R305: 10k, R_0402_1005Metric, B.Cu at (69.4, 36.8)
- added R306: 10k, R_0402_1005Metric, B.Cu at (71.6, 36.8)
- added R307: 10k, R_0402_1005Metric, B.Cu at (73.8, 36.8)
- added R308: 3.3k, R_0402_1005Metric, B.Cu at (76.0, 36.8)
- added R309: 3.3k, R_0402_1005Metric, B.Cu at (58.4, 6.21)
- added R31: 10, R_0402_1005Metric, B.Cu at (13.7, 12.8)
- added R310: 3.3k, R_0402_1005Metric, B.Cu at (62.0, 6.21)
- added R311: 10k, R_0402_1005Metric, B.Cu at (67.8, 6.21)
- added R312: 10k, R_0402_1005Metric, B.Cu at (72.6, 6.21)
- added R313: 10k, R_0402_1005Metric, B.Cu at (77.1, 6.21)
- added R320: 10, R_0402_1005Metric, B.Cu at (88.4, 29.3)
- added R321: 10, R_0402_1005Metric, B.Cu at (90.6, 29.3)
- added R322: 10, R_0402_1005Metric, B.Cu at (68.3, 35.0)
- added R323: 10, R_0402_1005Metric, B.Cu at (70.5, 35.0)
- added R324: 10, R_0402_1005Metric, B.Cu at (72.7, 35.0)
- added R325: 10, R_0402_1005Metric, B.Cu at (74.9, 35.0)
- added R326: 10k, R_0402_1005Metric, B.Cu at (77.1, 35.0)
- added R327: 10k, R_0402_1005Metric, B.Cu at (58.4, 36.8)
- added R328: 10k, R_0402_1005Metric, B.Cu at (60.6, 36.8)
- added R329: 10k, R_0402_1005Metric, B.Cu at (62.8, 36.8)
- added R330: 10k, R_0402_1005Metric, B.Cu at (65.0, 36.8)
- added R331: 10k, R_0402_1005Metric, B.Cu at (67.2, 36.8)
- added R332: 2.2, R_0603_1608Metric, B.Cu at (89.3, 27.3)
- added R333: 2.2, R_0603_1608Metric, B.Cu at (90.8, 6.28)
- added R334: 2.2, R_0603_1608Metric, B.Cu at (100.1, 17.3)
- added R335: 1mΩ 3W, R_2512_Shunt_Kelvin, F.Cu at (84.5, 4.40)
- added R40: 10, R_0402_1005Metric, B.Cu at (43.3, 33.0)
- added R400: 10k, R_0402_1005Metric, B.Cu at (34.2, 44.3)
- added R401: 10k DNP, R_0402_1005Metric, B.Cu at (36.4, 44.3)
- added R402: 100k, R_0402_1005Metric, B.Cu at (38.6, 44.3)
- added R403: 10k, R_0402_1005Metric, B.Cu at (40.8, 44.3)
- added R404: 1k, R_0402_1005Metric, B.Cu at (43.0, 44.3)
- added R405: 10k, R_0402_1005Metric, B.Cu at (37.3, 1.11)
- added R406: 10k, R_0402_1005Metric, B.Cu at (39.5, 1.11)
- added R407: 10k, R_0402_1005Metric, B.Cu at (41.7, 1.11)
- added R408: 3.3k, R_0402_1005Metric, B.Cu at (43.9, 1.11)
- added R409: 3.3k, R_0402_1005Metric, B.Cu at (46.1, 1.11)
- added R41: 10, R_0402_1005Metric, B.Cu at (45.5, 33.0)
- added R410: 3.3k, R_0402_1005Metric, B.Cu at (37.3, 2.40)
- added R411: 10k, R_0402_1005Metric, B.Cu at (39.5, 2.40)
- added R412: 10k, R_0402_1005Metric, B.Cu at (41.7, 2.40)
- added R413: 10k, R_0402_1005Metric, B.Cu at (43.9, 2.40)
- added R420: 10, R_0402_1005Metric, B.Cu at (55.7, 46.5)
- added R421: 10, R_0402_1005Metric, B.Cu at (57.9, 46.5)
- added R422: 10, R_0402_1005Metric, B.Cu at (34.2, 48.7)
- added R423: 10, R_0402_1005Metric, B.Cu at (36.4, 48.7)
- added R424: 10, R_0402_1005Metric, B.Cu at (38.6, 48.7)
- added R425: 10, R_0402_1005Metric, B.Cu at (40.8, 48.7)
- added R426: 10k, R_0402_1005Metric, B.Cu at (43.0, 48.7)
- added R427: 10k, R_0402_1005Metric, B.Cu at (45.2, 48.7)
- added R428: 10k, R_0402_1005Metric, B.Cu at (47.4, 48.7)
- added R429: 10k, R_0402_1005Metric, B.Cu at (49.6, 48.7)
- added R430: 10k, R_0402_1005Metric, B.Cu at (55.7, 48.7)
- added R431: 10k, R_0402_1005Metric, B.Cu at (57.9, 48.7)
- added R432: 2.2, R_0603_1608Metric, B.Cu at (45.7, 44.5)
- added R433: 2.2, R_0603_1608Metric, B.Cu at (49.0, 44.5)
- added R434: 2.2, R_0603_1608Metric, B.Cu at (52.3, 44.5)
- added R435: 1mΩ 3W, R_2512_Shunt_Kelvin, F.Cu at (32.9, 31.5)
- added R440: 4.7k, R_0603_1608Metric, B.Cu at (14.1, 22.9)
- added R441: 10k, R_0402_1005Metric, B.Cu at (16.9, 22.7)
- added R442: 100k, R_0402_1005Metric, B.Cu at (19.1, 22.7)
- added R443: 100k, R_0402_1005Metric, B.Cu at (21.3, 22.7)
- added R444: 47k, R_0402_1005Metric, B.Cu at (23.5, 22.7)
- added R50: 10, R_0402_1005Metric, B.Cu at (80.6, 6.62)
- added R51: 10, R_0402_1005Metric, B.Cu at (82.8, 6.62)
- added R60: 10, R_0402_1005Metric, B.Cu at (31.5, 20.6)
- added R61: 10, R_0402_1005Metric, B.Cu at (33.7, 20.6)
- added R80: 10k, R_0402_1005Metric, B.Cu at (73.8, 13.3)
- added R81: 10k, R_0402_1005Metric, B.Cu at (76.0, 13.3)
- added R82: 10k, R_0402_1005Metric, B.Cu at (58.4, 19.5)
- added R83: 330, R_0402_1005Metric, B.Cu at (78.1, 49.5)
- added SW1: RESET, SW_Push_1P1T_XKB_TS-1187A, F.Cu at (12.6, 13.0)
- added TH1: 10k NTC, R_0603_1608Metric, B.Cu at (26.2, 22.9)
- added TP1: +VDRV, TestPoint_Pad_D1.5mm, F.Cu at (13.6, 5.60)
- added TP10: DSHOT_L, TestPoint_Pad_D1.5mm, F.Cu at (102.5, 25.4)
- added TP2: +5V, TestPoint_Pad_D1.5mm, F.Cu at (10.8, 8.40)
- added TP200: ISENSE, TestPoint_Pad_D1.5mm, F.Cu at (36.7, 34.2)
- added TP201: VSENSE, TestPoint_Pad_D1.5mm, F.Cu at (39.4, 34.2)
- added TP202: TLM, TestPoint_Pad_D1.5mm, F.Cu at (42.2, 34.2)
- added TP203: I_L+, TestPoint_Pad_D1.5mm, F.Cu at (44.9, 34.2)
- added TP3: +3V3_A, TestPoint_Pad_D1.5mm, F.Cu at (5.20, 14.0)
- added TP4: +3V3_MCU, TestPoint_Pad_D1.5mm, F.Cu at (54.7, 38.9)
- added TP40: WEAPON_EN, TestPoint_Pad_D1.5mm, F.Cu at (44.5, 49.0)
- added TP5: GND, TestPoint_Pad_D1.5mm, F.Cu at (54.7, 41.6)
- added TP6: GND, TestPoint_Pad_D1.5mm, F.Cu at (41.7, 49.0)
- added U1: AP63205WU-7, TSOT-23-6, B.Cu at (63.2, 20.7)
- added U10: W25Q128JVSIQ, SOIC-8_5.3x5.3mm_P1.27mm, B.Cu at (65.8, 15.8)
- added U11: 74AHCT1G125GW, SOT-353_SC-70-5, B.Cu at (76.5, 47.6)
- added U2: AP2112K-3.3TRG1, SOT-23-5, B.Cu at (59.5, 2.25)
- added U20: AT32F421K8U7, QFN-32-1EP_5x5mm_P0.5mm_EP3.3x3.3mm, B.Cu at (39.2, 17.0)
- added U21: HX6288 / FD6288Q, QFN-24-1EP_4x4mm_P0.5mm_EP2.7x2.7mm, B.Cu at (45.8, 16.5)
- added U22: INA180A1, SOT-23-5, B.Cu at (51.4, 15.5)
- added U3: AP2112K-3.3TRG1, SOT-23-5, B.Cu at (74.2, 2.25)
- added U30: AT32F421K8U7, QFN-32-1EP_5x5mm_P0.5mm_EP3.3x3.3mm, B.Cu at (88.7, 22.9)
- added U31: HX6288 / FD6288Q, QFN-24-1EP_4x4mm_P0.5mm_EP2.7x2.7mm, B.Cu at (82.7, 12.3)
- added U32: INA180A1, SOT-23-5, B.Cu at (88.2, 11.4)
- added U4: INA226 0x40 pack, MSOP-10_3x3mm_P0.5mm, B.Cu at (51.6, 7.39)
- added U40: AT32F421K8U7, QFN-32-1EP_5x5mm_P0.5mm_EP3.3x3.3mm, B.Cu at (16.1, 31.1)
- added U41: HX6288 / FD6288Q, QFN-24-1EP_4x4mm_P0.5mm_EP2.7x2.7mm, B.Cu at (22.7, 30.6)
- added U42: INA180A1, SOT-23-5, B.Cu at (28.3, 29.7)
- added U5: INA226 0x41 L, MSOP-10_3x3mm_P0.5mm, B.Cu at (38.9, 34.3)
- added U6: INA226 0x44 R, MSOP-10_3x3mm_P0.5mm, B.Cu at (93.7, 12.0)
- added U7: INA226 0x45 W, MSOP-10_3x3mm_P0.5mm, B.Cu at (33.2, 16.6)
- added U8: LSM6DS3TR-C, LGA-14_3x2.5mm_P0.5mm_LayoutBorder3x4y, B.Cu at (59.2, 8.53)
- added U9: ADXL375BCCZ, LGA-14_3x5mm_P0.8mm_LayoutBorder1x6y, B.Cu at (67.4, 9.78)
Routing:
- net +5V: track 0.00 -> 281.6 mm, vias 0 -> 11
- net +3V3_MCU: track 0.00 -> 260.9 mm, vias 0 -> 15
- net +3V3_A: track 0.00 -> 252.4 mm, vias 0 -> 12
- net +VDRV: track 0.00 -> 235.3 mm, vias 0 -> 15
- net GND: track 0.00 -> 190.2 mm, vias 0 -> 183
- net +3V3_PICO: track 0.00 -> 158.4 mm, vias 0 -> 5
- net I2C1_SCL: track 0.00 -> 153.1 mm, vias 0 -> 8
- net I2C1_SDA: track 0.00 -> 148.9 mm, vias 0 -> 9
- net MOTOR_W_C: track 0.00 -> 126.1 mm, vias 0 -> 18
- net /Pico W and control I/O/RUN: track 0.00 -> 119.3 mm, vias 0 -> 4
- net MOTOR_W_B: track 0.00 -> 108.9 mm, vias 0 -> 17
- net /Pico W and control I/O/NTC_ADC: track 0.00 -> 107.3 mm, vias 0 -> 5
- net DSHOT_L: track 0.00 -> 87.5 mm, vias 0 -> 4
- net ARM_N: track 0.00 -> 86.1 mm, vias 0 -> 6
- net /ESC L control (AM32)/L_BEMF_B: track 0.00 -> 82.9 mm, vias 0 -> 6
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- added copper zone on F.Cu, net /ESC L power stage/I_L+
- added copper zone on F.Cu, net /ESC R power stage/I_R+
- added copper zone on F.Cu, net /ESC W power stage/I_W+
- added copper zone on B.Cu, net GND
- added copper zone on F.Cu, net GND
- added copper zone on In1.Cu, net GND
- added copper zone on F.Cu, net MOTOR_L_A
- added copper zone on F.Cu, net MOTOR_L_B
- added copper zone on F.Cu, net MOTOR_L_C
- added copper zone on F.Cu, net MOTOR_R_A
- added copper zone on F.Cu, net MOTOR_R_B
- added copper zone on F.Cu, net MOTOR_R_C
- added copper zone on F.Cu, net MOTOR_W_A
- added copper zone on F.Cu, net MOTOR_W_B
- added copper zone on F.Cu, net MOTOR_W_C
- added copper zone on B.Cu, net VBAT
- added copper zone on F.Cu, net VBAT
- added copper zone on In1.Cu, net VBAT
- added copper zone on B.Cu, net VBAT_PACK
- added copper zone on F.Cu, net VBAT_PACK
Other:
- board outline added: 104.5 x 51 mm
- copper layers 2 -> 4
- board text added: "ThumbsUp v1.2"
