File: hardware/kicad/thumbsup_esc_l.kicad_sch (KiCad schematic)
At the start: 32 parts, among them J20 SWD, U20 AT32F421K8U7, U21 HX6288 / FD6288Q, U22 INA180A1

Commit message: hardware: generated PCB layout pipeline (mech outline, placement, copper, Freerouting), rev v1.2
- tools/mech/chassis.py: Bambu 3MF -> PCB bay outline, boss positions, fit check
- tools/pcb/: board builder (netlist -> pcbnew), obstacle-aware placement with
  0 placement problems, power pours / via fields / gate and Kelvin stubs, pickup
  and GND vias, Freerouting DSN/SES driver, JLC fab outputs
- circuit: J4/C4/C426 dropped, motor holes between the FET rows, Kelvin net-ties
  in the shunt pad gap, M2.5 holes, SWD pad rows, fewer test points, I_x+ named
- docs: LAYOUT.md rewritten for the generated layout, PARTS/REQUIREMENTS/REVIEW
  updated; routing status recorded in LAYOUT.md section 5 (102 unconnected left,
  board is over-dense for a fully automatic finish)

Co-Authored-By: Claude Fable 5.1 <noreply@anthropic.com>
Parts:
- J20: footprint Connector_PinHeader_2.54mm:PinHeader_1x05_P2.54mm_Vertical -> thumbsup:SWD_1x05_P1.27mm_Pads; Note 3V3 SWDIO SWCLK NRST GND -> 1.27 mm pads: 3V3 SWDIO SWCLK NRST GND
