File: hardware/kicad/thumbsup_esc_l_bridge.kicad_sch (KiCad schematic)
At the start: 35 parts, among them J21 MOTOR L, Q20 HYG015N04LS1C2, Q21 HYG015N04LS1C2, Q22 HYG015N04LS1C2, Q23 HYG015N04LS1C2, Q24 HYG015N04LS1C2, Q25 HYG015N04LS1C2

Commit message: hardware: generated PCB layout pipeline (mech outline, placement, copper, Freerouting), rev v1.2
- tools/mech/chassis.py: Bambu 3MF -> PCB bay outline, boss positions, fit check
- tools/pcb/: board builder (netlist -> pcbnew), obstacle-aware placement with
  0 placement problems, power pours / via fields / gate and Kelvin stubs, pickup
  and GND vias, Freerouting DSN/SES driver, JLC fab outputs
- circuit: J4/C4/C426 dropped, motor holes between the FET rows, Kelvin net-ties
  in the shunt pad gap, M2.5 holes, SWD pad rows, fewer test points, I_x+ named
- docs: LAYOUT.md rewritten for the generated layout, PARTS/REQUIREMENTS/REVIEW
  updated; routing status recorded in LAYOUT.md section 5 (102 unconnected left,
  board is over-dense for a fully automatic finish)

Co-Authored-By: Claude Fable 5.1 <noreply@anthropic.com>
Parts:
- J21: footprint thumbsup:MotorPads_1x03_P5.00mm -> thumbsup:MotorHoles_1x03_P5.90mm; Note 2 mm holes + 4x3 lands, 30 A -> 3x 2 mm plated holes in the phase pours, 30 A
- NT20: footprint NetTie:NetTie-2_SMD_Pad0.5mm -> thumbsup:NetTie-2_Kelvin_0.4mm; Note on shunt pad 1 -> in the shunt pad gap
- NT21: footprint NetTie:NetTie-2_SMD_Pad0.5mm -> thumbsup:NetTie-2_Kelvin_0.4mm; Note on shunt pad 2 -> in the shunt pad gap
Connections:
- net I_L+: now reaches NT20.1, Q21.1 (S), Q21.2 (S), Q21.3 (S), Q23.1 (S), Q23.2 (S), Q23.3 (S), Q25.1 (S), Q25.2 (S), Q25.3 (S), R227.2, R229.2, R231.2, R235.1, TP203.1
