File: hardware/kicad/thumbsup_esc_r.kicad_sch (KiCad schematic)
At the start: 32 parts, among them J30 SWD, U30 AT32F421K8U7, U31 HX6288 / FD6288Q, U32 INA180A1

Commit message: hardware: generated PCB layout pipeline (mech outline, placement, copper, Freerouting), rev v1.2
- tools/mech/chassis.py: Bambu 3MF -> PCB bay outline, boss positions, fit check
- tools/pcb/: board builder (netlist -> pcbnew), obstacle-aware placement with
  0 placement problems, power pours / via fields / gate and Kelvin stubs, pickup
  and GND vias, Freerouting DSN/SES driver, JLC fab outputs
- circuit: J4/C4/C426 dropped, motor holes between the FET rows, Kelvin net-ties
  in the shunt pad gap, M2.5 holes, SWD pad rows, fewer test points, I_x+ named
- docs: LAYOUT.md rewritten for the generated layout, PARTS/REQUIREMENTS/REVIEW
  updated; routing status recorded in LAYOUT.md section 5 (102 unconnected left,
  board is over-dense for a fully automatic finish)

Co-Authored-By: Claude Fable 5.1 <noreply@anthropic.com>
Parts:
- removed TP300: ISENSE, TestPoint:TestPoint_Pad_D1.5mm, symbol Connector:TestPoint
- removed TP301: VSENSE, TestPoint:TestPoint_Pad_D1.5mm, symbol Connector:TestPoint
- removed TP302: TLM, TestPoint:TestPoint_Pad_D1.5mm, symbol Connector:TestPoint
- J30: footprint Connector_PinHeader_2.54mm:PinHeader_1x05_P2.54mm_Vertical -> thumbsup:SWD_1x05_P1.27mm_Pads; Note 3V3 SWDIO SWCLK NRST GND -> 1.27 mm pads: 3V3 SWDIO SWCLK NRST GND
Connections:
- net R_TLM: no longer names the net of U30.29 (PB6_TLM_TX)
- no-connect marks 15 -> 16
Other:
- note removed: "Test points (PB6 = AM32 KISS telemetry, 115200)"
