File: hardware/kicad/thumbsup_esc_r_bridge.kicad_sch (KiCad schematic)
At the start: 35 parts, among them J31 MOTOR R, Q30 HYG015N04LS1C2, Q31 HYG015N04LS1C2, Q32 HYG015N04LS1C2, Q33 HYG015N04LS1C2, Q34 HYG015N04LS1C2, Q35 HYG015N04LS1C2

Commit message: hardware: generated PCB layout pipeline (mech outline, placement, copper, Freerouting), rev v1.2
- tools/mech/chassis.py: Bambu 3MF -> PCB bay outline, boss positions, fit check
- tools/pcb/: board builder (netlist -> pcbnew), obstacle-aware placement with
  0 placement problems, power pours / via fields / gate and Kelvin stubs, pickup
  and GND vias, Freerouting DSN/SES driver, JLC fab outputs
- circuit: J4/C4/C426 dropped, motor holes between the FET rows, Kelvin net-ties
  in the shunt pad gap, M2.5 holes, SWD pad rows, fewer test points, I_x+ named
- docs: LAYOUT.md rewritten for the generated layout, PARTS/REQUIREMENTS/REVIEW
  updated; routing status recorded in LAYOUT.md section 5 (102 unconnected left,
  board is over-dense for a fully automatic finish)

Co-Authored-By: Claude Fable 5.1 <noreply@anthropic.com>
Parts:
- removed TP303: I_R+, TestPoint:TestPoint_Pad_D1.5mm, symbol Connector:TestPoint
- J31: footprint thumbsup:MotorPads_1x03_P5.00mm -> thumbsup:MotorHoles_1x03_P5.90mm; Note 2 mm holes + 4x3 lands, 30 A -> 3x 2 mm plated holes in the phase pours, 30 A
- NT30: footprint NetTie:NetTie-2_SMD_Pad0.5mm -> thumbsup:NetTie-2_Kelvin_0.4mm; Note on shunt pad 1 -> in the shunt pad gap
- NT31: footprint NetTie:NetTie-2_SMD_Pad0.5mm -> thumbsup:NetTie-2_Kelvin_0.4mm; Note on shunt pad 2 -> in the shunt pad gap
Connections:
- net I_R+: now reaches NT30.1, Q31.1 (S), Q31.2 (S), Q31.3 (S), Q33.1 (S), Q33.2 (S), Q33.3 (S), Q35.1 (S), Q35.2 (S), Q35.3 (S), R327.2, R329.2, R331.2, R335.1
