File: hardware/kicad/thumbsup_esc_w_bridge.kicad_sch (KiCad schematic)
At the start: 36 parts, among them J41 MOTOR W, Q40 HYG015N04LS1C2, Q41 HYG015N04LS1C2, Q42 HYG015N04LS1C2, Q43 HYG015N04LS1C2, Q44 HYG015N04LS1C2, Q45 HYG015N04LS1C2

Commit message: hardware: generated PCB layout pipeline (mech outline, placement, copper, Freerouting), rev v1.2
- tools/mech/chassis.py: Bambu 3MF -> PCB bay outline, boss positions, fit check
- tools/pcb/: board builder (netlist -> pcbnew), obstacle-aware placement with
  0 placement problems, power pours / via fields / gate and Kelvin stubs, pickup
  and GND vias, Freerouting DSN/SES driver, JLC fab outputs
- circuit: J4/C4/C426 dropped, motor holes between the FET rows, Kelvin net-ties
  in the shunt pad gap, M2.5 holes, SWD pad rows, fewer test points, I_x+ named
- docs: LAYOUT.md rewritten for the generated layout, PARTS/REQUIREMENTS/REVIEW
  updated; routing status recorded in LAYOUT.md section 5 (102 unconnected left,
  board is over-dense for a fully automatic finish)

Co-Authored-By: Claude Fable 5.1 <noreply@anthropic.com>
Parts:
- removed C426: 470u 25V hybrid, Capacitor_SMD:CP_Elec_10x10.5, symbol Device:C_Polarized
- removed TP403: I_W+, TestPoint:TestPoint_Pad_D1.5mm, symbol Connector:TestPoint
- C425: value 470u 25V hybrid -> 470u 25V polymer 4A; footprint Capacitor_SMD:CP_Elec_10x10.5 -> Capacitor_SMD:CP_Elec_10x12.5; LCSC C242138 -> C46528073; Note EEHZK1E471P 20 mOhm, glue -> KNSCHA 118EC421 14 mOhm / 4 A; alt EEHZK1E471P C242138
- J41: footprint thumbsup:MotorPads_1x03_P5.00mm -> thumbsup:MotorHoles_1x03_P5.90mm; Note 2 mm holes + 4x3 lands, 30 A -> 3x 2 mm plated holes in the phase pours, 30 A
- NT40: footprint NetTie:NetTie-2_SMD_Pad0.5mm -> thumbsup:NetTie-2_Kelvin_0.4mm; Note on shunt pad 1 -> in the shunt pad gap
- NT41: footprint NetTie:NetTie-2_SMD_Pad0.5mm -> thumbsup:NetTie-2_Kelvin_0.4mm; Note on shunt pad 2 -> in the shunt pad gap
Connections:
- net I_W+: now reaches NT40.1, Q41.1 (S), Q41.2 (S), Q41.3 (S), Q43.1 (S), Q43.2 (S), Q43.3 (S), Q45.1 (S), Q45.2 (S), Q45.3 (S), R427.2, R429.2, R431.2, R435.1
