File: hardware/kicad/thumbsup_pack.kicad_sch (KiCad schematic)
At the start: 21 parts, among them J1 XT30PW-M, J4 POWER LINK, Q1 AP40P05

Commit message: hardware: generated PCB layout pipeline (mech outline, placement, copper, Freerouting), rev v1.2
- tools/mech/chassis.py: Bambu 3MF -> PCB bay outline, boss positions, fit check
- tools/pcb/: board builder (netlist -> pcbnew), obstacle-aware placement with
  0 placement problems, power pours / via fields / gate and Kelvin stubs, pickup
  and GND vias, Freerouting DSN/SES driver, JLC fab outputs
- circuit: J4/C4/C426 dropped, motor holes between the FET rows, Kelvin net-ties
  in the shunt pad gap, M2.5 holes, SWD pad rows, fewer test points, I_x+ named
- docs: LAYOUT.md rewritten for the generated layout, PARTS/REQUIREMENTS/REVIEW
  updated; routing status recorded in LAYOUT.md section 5 (102 unconnected left,
  board is over-dense for a fully automatic finish)

Co-Authored-By: Claude Fable 5.1 <noreply@anthropic.com>
Parts:
- removed C4: 470u 25V hybrid, Capacitor_SMD:CP_Elec_10x10.5, symbol Device:C_Polarized
- removed H4: M3, MountingHole:MountingHole_3.2mm_M3, symbol Mechanical:MountingHole
- removed J4: POWER LINK, Connector_AMASS:AMASS_XT30PW-M_1x02_P2.50mm_Horizontal, symbol Connector:Conn_01x02_Pin
- H1, H2, H3: value M3 -> M2.5; footprint MountingHole:MountingHole_3.2mm_M3 -> MountingHole:MountingHole_2.7mm_M2.5
- NT1: footprint NetTie:NetTie-2_SMD_Pad0.5mm -> thumbsup:NetTie-2_Kelvin_0.4mm; Note on R2 pad 1 -> in the R2 pad gap
- NT2: footprint NetTie:NetTie-2_SMD_Pad0.5mm -> thumbsup:NetTie-2_Kelvin_0.4mm; Note on R2 pad 2 -> in the R2 pad gap
Connections:
- net VBAT_PACK: now also NT1.1, R2.1
Other:
- note added: "J1 is the SPARC disconnect (PWR-2): mates through a slot in the back wall"
- note added: "Mechanical: 3x M2.5 mounting holes (positions from tools/mech/chassis.py), 3 fiducials"
- note added: "Pack input: XT30 → TVS/filter → 1 mΩ shunt (Kelvin net-ties) → VBAT (bridges) ; VBAT → P-FET reverse-polarity → +VDRV (logic)"
- note removed: "J4 POWER LINK = SPARC disconnect (PWR-2)"
- note removed: "Mechanical: 4x M3 mounting holes, 3 fiducials (positions from the chassis in layout)"
- note removed: "Pack input: XT30 → TVS/filter → POWER LINK J4 → 1 mΩ shunt (Kelvin net-ties) → VBAT (bridges) ; VBAT → P-FET reverse-polarity → +VDRV (logic)"
