File: hardware/kicad/thumbsup_pico.kicad_sch (KiCad schematic)
At the start: 21 parts, among them J2 ARM link, J3 EXPANSION, SW1 RESET

Commit message: hardware: generated PCB layout pipeline (mech outline, placement, copper, Freerouting), rev v1.2
- tools/mech/chassis.py: Bambu 3MF -> PCB bay outline, boss positions, fit check
- tools/pcb/: board builder (netlist -> pcbnew), obstacle-aware placement with
  0 placement problems, power pours / via fields / gate and Kelvin stubs, pickup
  and GND vias, Freerouting DSN/SES driver, JLC fab outputs
- circuit: J4/C4/C426 dropped, motor holes between the FET rows, Kelvin net-ties
  in the shunt pad gap, M2.5 holes, SWD pad rows, fewer test points, I_x+ named
- docs: LAYOUT.md rewritten for the generated layout, PARTS/REQUIREMENTS/REVIEW
  updated; routing status recorded in LAYOUT.md section 5 (102 unconnected left,
  board is over-dense for a fully automatic finish)

Co-Authored-By: Claude Fable 5.1 <noreply@anthropic.com>
Parts:
- removed TP11: DSHOT_R, TestPoint:TestPoint_Pad_D1.5mm, symbol Connector:TestPoint
- removed TP12: DSHOT_W, TestPoint:TestPoint_Pad_D1.5mm, symbol Connector:TestPoint
- removed TP13: I2C1_SDA, TestPoint:TestPoint_Pad_D1.5mm, symbol Connector:TestPoint
- removed TP14: I2C1_SCL, TestPoint:TestPoint_Pad_D1.5mm, symbol Connector:TestPoint
- removed TP15: ARM_N, TestPoint:TestPoint_Pad_D1.5mm, symbol Connector:TestPoint
- TP10: Note (none) -> I2C/ARM/DSHOT_R/W are on J3, J2 and the AT32 pads
Other:
- note added: "Test point"
- note removed: "Test points"
