File: hardware/motor_board/kicad/motor_board/power.kicad_sch (KiCad schematic)
At the start: 44 parts, among them J4 S5B-XH-A, Q7 HYG015N04LS1C2, Q8 HYG015N04LS1C2, U13 LM74502DDFR, U7 INA239AIDGSR, U8 BQ76907RGRR

Commit message: v2 package swaps (rev L2), after adversarial review: U6 WQFN-14 (EP to GND), D2 PMEG4030ER, L1 ZEMS404030 4.1 mm, J4 vertical XH, J2/J3 genuine JST vertical SH, R300/R400 0603 anti-surge, R15/C14/D10 one size down; drive VM bulk 2 x 10 uF X7R 1210 per drive (C309/C310/C409/C410 removed, user OK) - the 1206 X5R kept only ~2.3 uF at 16.8 V
sim_hotplug.py models MLCC DC bias (worst bounce 2.14 V/us at 0 C, 2.62 at -40 C); library check 0 errors, mutation test all caught; schematic regenerated, nets 176/176; v2 board rebuilt: DRC 0, parity 0; WQFN-14 3D model generated; DESIGN/calcs/BOM/FAB/CHANGES updated (CPL rotation fix for J2/J3/J4)

Co-Authored-By: Claude Opus 5.5 (1M context) <noreply@anthropic.com>
Parts:
- removed D10: 1N4148W, Diode_SMD:D_SOD-123, symbol motor_board:1N4148W
- removed J4: S5B-XH-A, Connector_JST:JST_XH_S5B-XH-A_1x05_P2.50mm_Horizontal, symbol motor_board:S5B-XH-A
- added D10: 1N4148WS, Diode_SMD:D_SOD-323, symbol motor_board:1N4148WS
- added J4: B5B-XH-A, Connector_JST:JST_XH_B5B-XH-A_1x05_P2.50mm_Vertical, symbol motor_board:B5B-XH-A
- C14: footprint Capacitor_SMD:C_0805_2012Metric -> Capacitor_SMD:C_0603_1608Metric; LCSC C28233 -> C15725
- R15: value 6.8k 0805 -> 6.8k 0603; footprint Resistor_SMD:R_0805_2012Metric -> Resistor_SMD:R_0603_1608Metric; LCSC C17772 -> C23212
Connections:
- net BAL0: now also J4.1 (Pin_1)
- net BAL1: now also J4.2 (Pin_2)
- net BAL2: now also J4.3 (Pin_3)
- net BAL3: now also J4.4 (Pin_4)
- net BAL4: now also J4.5 (Pin_5)
- net PSW_DV: now also D10.1 (K)
- net PSW_RG: now also D10.2 (A)
Changed lines of the file:
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@@
 	)
 	(symbol
-		(lib_id "motor_board:1N4148W")
+		(lib_id "motor_board:1N4148WS")
 		(at 99.06 124.46 0)
 		(unit 1)
@@
 			)
 		)
-		(property "Value" "1N4148W"
+		(property "Value" "1N4148WS"
 			(at 99.06 127 0)
 			(effects
@@
 			)
 		)
-		(property "Footprint" "Diode_SMD:D_SOD-123"
+		(property "Footprint" "Diode_SMD:D_SOD-323"
 			(at 99.06 128.905 0)
 			(hide yes)
@@
 			)
 		)
-		(property "Datasheet" "https://www.lcsc.com/product-detail/C81598.html"
+		(property "Datasheet" "https://www.lcsc.com/product-detail/C2128.html"
 			(at 99.06 124.46 0)
 			(hide yes)
@@
 			)
 		)
-		(property "Description" "Switching diode 75 V 150 mA, SOD-123"
+		(property "Description" "Switching diode 100 V 150 mA, SOD-323"
 			(at 99.06 124.46 0)
 			(hide yes)
@@
 			)
 		)
-		(property "LCSC" "C81598"
+		(property "LCSC" "C2128"
 			(at 99.06 124.46 0)
 			(hide yes)
@@
 			)
 		)
-		(property "MPN" "1N4148W"
+		(property "MPN" "1N4148WS"
 			(at 99.06 124.46 0)
 			(hide yes)
@@
 			)
 		)
-		(property "Footprint" "Capacitor_SMD:C_0805_2012Metric"
+		(property "Footprint" "Capacitor_SMD:C_0603_1608Metric"
 			(at 69.5452 168.91 0)
 			(hide yes)
@@
 			)
 		)
-		(property "LCSC" "C28233"
+		(property "LCSC" "C15725"
 			(at 68.58 165.1 0)
 			(hide yes)
@@
 	)
 	(symbol
-		(lib_id "motor_board:S5B-XH-A")
+		(lib_id "motor_board:B5B-XH-A")
 		(at 198.12 96.52 0)
 		(unit 1)
@@
 			)
 		)
-		(property "Value" "S5B-XH-A"
+		(property "Value" "B5B-XH-A"
 			(at 198.12 104.14 0)
 			(effects
@@
 			)
 		)
-		(property "Footprint" "Connector_JST:JST_XH_S5B-XH-A_1x05_P2.50mm_Horizontal"
+		(property "Footprint" "Connector_JST:JST_XH_B5B-XH-A_1x05_P2.50mm_Vertical"
 			(at 198.12 96.52 0)
 			(hide yes)
@@
 			)
 		)
-		(property "Datasheet" "https://www.lcsc.com/product-detail/C263757.html"
+		(property "Datasheet" "https://www.lcsc.com/product-detail/C157991.html"
 			(at 198.12 96.52 0)
 			(hide yes)
@@
 			)
 		)
-		(property "Description" "JST XH 5-pin side-entry THT (balance lead)"
+		(property "Description" "JST XH 5-pin vertical THT (balance lead), 9.8 mm mated"
 			(at 198.12 96.52 0)
 			(hide yes)
@@
 			)
 		)
-		(property "LCSC" "C263757"
+		(property "LCSC" "C157991"
 			(at 198.12 96.52 0)
 			(hide yes)
@@
 			)
 		)
-		(property "MPN" "S5B-XH-A"
+		(property "MPN" "B5B-XH-A"
 			(at 198.12 96.52 0)
 			(hide yes)
@@
 			)
 		)
-		(property "Value" "6.8k 0805"
+		(property "Value" "6.8k 0603"
 			(at 355.6 104.14 90)
 			(effects
@@
 			)
 		)
-		(property "Footprint" "Resistor_SMD:R_0805_2012Metric"
+		(property "Footprint" "Resistor_SMD:R_0603_1608Metric"
 			(at 353.822 104.14 90)
 			(hide yes)
@@
 			)
 		)
-		(property "LCSC" "C17772"
+		(property "LCSC" "C23212"
 			(at 355.6 104.14 0)
 			(hide yes)

Commit message: Schematic regenerated for C117 + U7 INA239AQDGSRQ1 (lib_build parts/symbol, SHEETS/blocks); board sync stage hR (tail_apply op 'sync' via schsync.py: footprints re-linked to the new symbol UUIDs, U7 fields, C117 added provisionally near U8 and routed); r2/pourtest.py power-net pour acceptance test (12 nets failing on hF: the rework list); DRC 0, parity 0
Co-Authored-By: Claude Opus 5.5 (1M context) <noreply@anthropic.com>
Parts:
- removed U7: INA239AIDGSR, Package_SO:MSOP-10_3x3mm_P0.5mm, symbol motor_board:INA239AIDGSR
- added C117: 100nF 50V, Capacitor_SMD:C_0603_1608Metric, symbol Device:C
- added U7: INA239AQDGSRQ1, Package_SO:MSOP-10_3x3mm_P0.5mm, symbol motor_board:INA239AQDGSRQ1
Connections:
- net +3V3: now also U7.6 (VS)
- net BMS_BAT: now also C117.1
- net GND: now also C117.2, U7.7 (GND)
- net INA_INN: now also U7.9 (IN-)
- net INA_INP: now also U7.10 (IN+)
- net INA_nCS: now also U7.1 (~{CS})
- net SPI_MISO: now also U7.4 (MISO)
- net SPI_MOSI: now also U7.2 (MOSI)
- net SPI_SCK: now also U7.5 (SCLK)
- net VBAT: now also U7.8 (VBUS)
- net W_nFAULT: now also U7.3 (~{ALERT})
