File: hardware/motor_board/kicad/motor_board/sensors.kicad_sch (KiCad schematic)
At the start: 40 parts, among them J2 WAFER-SH1.0-6PWB, J3 WAFER-SH1.0-6PWB, U10 SN74LVC3G17DCUR, U11 TPS22945DCKR, U12 TPS22945DCKR, U9 SN74LVC3G17DCUR

Commit message: v2 package swaps (rev L2), after adversarial review: U6 WQFN-14 (EP to GND), D2 PMEG4030ER, L1 ZEMS404030 4.1 mm, J4 vertical XH, J2/J3 genuine JST vertical SH, R300/R400 0603 anti-surge, R15/C14/D10 one size down; drive VM bulk 2 x 10 uF X7R 1210 per drive (C309/C310/C409/C410 removed, user OK) - the 1206 X5R kept only ~2.3 uF at 16.8 V
sim_hotplug.py models MLCC DC bias (worst bounce 2.14 V/us at 0 C, 2.62 at -40 C); library check 0 errors, mutation test all caught; schematic regenerated, nets 176/176; v2 board rebuilt: DRC 0, parity 0; WQFN-14 3D model generated; DESIGN/calcs/BOM/FAB/CHANGES updated (CPL rotation fix for J2/J3/J4)

Co-Authored-By: Claude Opus 5.5 (1M context) <noreply@anthropic.com>
Parts:
- removed J2, J3: WAFER-SH1.0-6PWB, motor_board:SH1.0-6P_RA_XUNPU_WAFER-SH1.0-6PWB, symbol motor_board:WAFER-SH1.0-6PWB
- added J2, J3: BM06B-SRSS-TB, Connector_JST:JST_SH_BM06B-SRSS-TB_1x06-1MP_P1.00mm_Vertical, symbol motor_board:BM06B-SRSS-TB
Connections:
- net GND: now also J2.2 (Pin_2), J2.MP (MountPin), J3.2 (Pin_2), J3.MP (MountPin)
- net L_H1: now also J2.3 (Pin_3)
- net L_H2: now also J2.4 (Pin_4)
- net L_H3: now also J2.5 (Pin_5)
- net L_TEMPJ: now also J2.6 (Pin_6)
- net L_VS: now also J2.1 (Pin_1)
- net R_H1: now also J3.3 (Pin_3)
- net R_H2: now also J3.4 (Pin_4)
- net R_H3: now also J3.5 (Pin_5)
- net R_TEMPJ: now also J3.6 (Pin_6)
- net R_VS: now also J3.1 (Pin_1)
